File: hardware/P1_Lock.kicad_sch (KiCad schematic)
At the start: 5 parts, among them J1 Conn_01x07, U1 STM32L476RGTx, U2 NHD-0420H1Z

Commit message: Partial Wiring
Connections:
- net at D1.1 (K): now also U1.18 (VSS), U1.31 (VSS), U1.47 (VSS), U1.63 (VSS)
- net at D1.2 (A): now also R1.1
- net at J1.1 (Pin_1): now also U1.21 (PA5)
- net at J1.2 (Pin_2): now also U1.22 (PA6)
- net at J1.3 (Pin_3): now also U1.23 (PA7)
- net at U1.20 (PA4): now also R1.2
Other:
- moved on the sheet: D1, R1
Changed lines of the file:
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@@
 		(title "P1 Lock Wiring Schematic")
+	)
+	(wire
+		(pts
+			(xy 144.78 67.31) (xy 160.02 67.31)
+		)
+		(stroke
+			(width 0)
+			(type default)
+		)
+	)
+	(wire
+		(pts
+			(xy 175.26 64.77) (xy 175.26 151.13)
+		)
+		(stroke
+			(width 0)
+			(type default)
+		)
+	)
+	(wire
+		(pts
+			(xy 144.78 64.77) (xy 157.48 64.77)
+		)
+		(stroke
+			(width 0)
+			(type default)
+		)
+	)
+	(wire
+		(pts
+			(xy 127 151.13) (xy 127 143.51)
+		)
+		(stroke
+			(width 0)
+			(type default)
+		)
+	)
+	(wire
+		(pts
+			(xy 144.78 69.85) (xy 157.48 69.85)
+		)
+		(stroke
+			(width 0)
+			(type default)
+		)
+	)
+	(wire
+		(pts
+			(xy 165.1 64.77) (xy 167.64 64.77)
+		)
+		(stroke
+			(width 0)
+			(type default)
+		)
+	)
+	(wire
+		(pts
+			(xy 175.26 151.13) (xy 127 151.13)
+		)
+		(stroke
+			(width 0)
+			(type default)
+		)
+	)
+	(wire
+		(pts
+			(xy 157.48 110.49) (xy 157.48 69.85)
+		)
+		(stroke
+			(width 0)
+			(type default)
+		)
+	)
+	(wire
+		(pts
+			(xy 154.94 72.39) (xy 144.78 72.39)
+		)
+		(stroke
+			(width 0)
+			(type default)
+		)
+	)
+	(wire
+		(pts
+			(xy 187.96 107.95) (xy 160.02 107.95)
+		)
+		(stroke
+			(width 0)
+			(type default)
+		)
+	)
+	(wire
+		(pts
+			(xy 187.96 110.49) (xy 157.48 110.49)
+		)
+		(stroke
+			(width 0)
+			(type default)
+		)
+	)
+	(wire
+		(pts
+			(xy 154.94 113.03) (xy 187.96 113.03)
+		)
+		(stroke
+			(width 0)
+			(type default)
+		)
+	)
+	(wire
+		(pts
+			(xy 154.94 113.03) (xy 154.94 72.39)
+		)
+		(stroke
+			(width 0)
+			(type default)
+		)
+	)
+	(wire
+		(pts
+			(xy 160.02 67.31) (xy 160.02 107.95)
+		)
+		(stroke
+			(width 0)
+			(type default)
+		)
 	)
 	(symbol
 		(lib_id "Device:LED")
-		(at 165.1 66.04 0)
+		(at 171.45 63.5 0)
 		(unit 1)
 		(body_style 1)
@@
 		(fields_autoplaced yes)
 		(property "Reference" "D1"
-			(at 163.5125 59.69 0)
+			(at 169.8625 57.15 0)
 			(show_name no)
 			(do_not_autoplace no)
@@
 		)
 		(property "Value" "LED"
-			(at 163.5125 62.23 0)
+			(at 169.8625 59.69 0)
 			(show_name no)
 			(do_not_autoplace no)
@@
 		)
 		(property "Footprint" ""
-			(at 165.1 66.04 0)
+			(at 171.45 63.5 0)
 			(hide yes)
 			(show_name no)
@@
 		)
 		(property "Datasheet" ""
-			(at 165.1 66.04 0)
+			(at 171.45 63.5 0)
 			(hide yes)
 			(show_name no)
@@
 		)
 		(property "Description" "Light emitting diode"
-			(at 165.1 66.04 0)
+			(at 171.45 63.5 0)
 			(hide yes)
 			(show_name no)
@@
 		)
 		(property "Sim.Pins" "1=K 2=A"
-			(at 165.1 66.04 0)
+			(at 171.45 64.77 0)
 			(hide yes)
 			(show_name no)
@@
 		(pin "64"
 		)
+		(pin "65"
+		)
 		(instances
 			(project "P1_Lock"
@@
 	(symbol
 		(lib_id "Device:R")
-		(at 165.1 78.74 0)
+		(at 161.29 64.77 0)
 		(unit 1)
 		(body_style 1)
@@
 		(fields_autoplaced yes)
 		(property "Reference" "R1"
-			(at 167.64 77.4699 0)
+			(at 160.274 62.738 0)
 			(show_name no)
 			(do_not_autoplace no)
@@
 		)
 		(property "Value" "R"
-			(at 167.64 80.0099 0)
+			(at 160.782 66.802 0)
 			(show_name no)
 			(do_not_autoplace no)
@@
 		)
 		(property "Footprint" ""
-			(at 163.322 78.74 90)
+			(at 159.512 64.77 90)
 			(hide yes)
 			(show_name no)
@@
 		)
 		(property "Datasheet" ""
-			(at 165.1 78.74 0)
+			(at 161.29 64.77 0)
 			(hide yes)
 			(show_name no)
@@
 		)
 		(property "Description" "Resistor"
-			(at 165.1 78.74 0)
-			(hide yes)
-			(show_name no)
+			(at 161.29 64.77 0)
+			(hide yes)
+			(show_name no)

Commit message: replaced the LCD with our local schematic
Parts:
- removed U2: NHD-0420H1Z, Display:NHD-0420H1Z, symbol Display_Character:NHD-0420H1Z
- added DS1: QAPASS 1602A, Package_QFP:TQFP-100_14x14mm_P0.5mm, symbol P1_SymbolLibrary:QAPASS 1602A
Changed lines of the file:
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@@
+	)
+	(symbol
+		(lib_id "P1_SymbolLibrary:QAPASS 1602A")
+		(at 198.12 71.12 0)
+		(unit 1)
+		(body_style 1)
+		(exclude_from_sim no)
+		(in_bom yes)
+		(on_board yes)
+		(in_pos_files yes)
+		(dnp no)
+		(fields_autoplaced yes)
+		(property "Reference" "DS1"
+			(at 200.2633 48.26 0)
+			(show_name no)
+			(do_not_autoplace no)
+			(effects
+				(font
+					(size 1.27 1.27)
+				)
+				(justify left)
+			)
+		)
+		(property "Value" "QAPASS 1602A"
+			(at 200.2633 50.8 0)
+			(show_name no)
+			(do_not_autoplace no)
+			(effects
+				(font
+					(size 1.27 1.27)
+				)
+				(justify left)
+			)
+		)
+		(property "Footprint" "Package_QFP:TQFP-100_14x14mm_P0.5mm"
+			(at 198.12 71.12 0)
+			(hide yes)
+			(show_name no)
+			(do_not_autoplace no)
+			(effects
+				(font
+					(size 1.27 1.27)
+				)
+			)
+		)
+		(property "Datasheet" ""
+			(at 198.12 71.12 0)
+			(hide yes)
+			(show_name no)
+			(do_not_autoplace no)
+			(effects
+				(font
+					(size 1.27 1.27)
+				)
+			)
+		)
+		(property "Description" "16x2 character LCD module, HD44780-compatible"
+			(at 198.12 71.12 0)
+			(hide yes)
+			(show_name no)
+			(do_not_autoplace no)
+			(effects
+				(font
+					(size 1.27 1.27)
+				)
+			)
+		)
+		(pin "14"
+		)
+		(pin "15"
+		)
+		(pin "9"
+		)
+		(pin "2"
+		)
+		(pin "3"
+		)
+		(pin "7"
+		)
+		(pin "12"
+		)
+		(pin "4"
+		)
+		(pin "1"
+		)
+		(pin "16"
+		)
+		(pin "13"
+		)
+		(pin "11"
+		)
+		(pin "8"
+		)
+		(pin "10"
+		)
+		(pin "5"
+		)
+		(pin "6"
+		)
+		(instances
+			(project "P1_Lock"
+				(path "/5e2df9ca-03bb-49be-9c86-c051a8edf5f2"
+					(reference "DS1")
+					(unit 1)
+				)
+			)
+		)
 	)
 	(symbol
@@
 					(unit 1)
 				)
-			)
-		)
-	)
-	(symbol
-		(lib_id "Display_Character:NHD-0420H1Z")
-		(at 198.12 66.04 0)
-		(unit 1)
-		(body_style 1)
-		(exclude_from_sim no)
-		(in_bom yes)
-		(on_board yes)
-		(in_pos_files yes)
-		(dnp no)
-		(fields_autoplaced yes)
-		(property "Reference" "U2"
-			(at 200.2633 86.36 0)
-			(show_name no)
-			(do_not_autoplace no)
-			(effects
-				(font
-					(size 1.27 1.27)
-				)
-				(justify left)
-			)
-		)
-		(property "Value" "NHD-0420H1Z"
-			(at 200.2633 88.9 0)
-			(show_name no)
-			(do_not_autoplace no)
-			(effects
-				(font
-					(size 1.27 1.27)
-				)
-				(justify left)
-			)
-		)
-		(property "Footprint" "Display:NHD-0420H1Z"
-			(at 198.12 88.9 0)
-			(hide yes)
-			(show_name no)
-			(do_not_autoplace no)
-			(effects
-				(font
-					(size 1.27 1.27)
-				)
-			)
-		)
-		(property "Datasheet" "http://www.newhavendisplay.com/specs/NHD-0420H1Z-FSW-GBW-33V3.pdf"
-			(at 200.66 68.58 0)
-			(hide yes)
-			(show_name no)
-			(do_not_autoplace no)
-			(effects
-				(font
-					(size 1.27 1.27)
-				)
-			)
-		)
-		(property "Description" "LCD 20x4 Alphanumeric 16pin Blue/White/Green Backlight, 8bit parallel, 3.3V VDD"
-			(at 198.12 66.04 0)
-			(hide yes)
-			(show_name no)
-			(do_not_autoplace no)
-			(effects
-				(font
-					(size 1.27 1.27)
-				)
-			)
-		)
-		(pin "10"
-		)
-		(pin "6"
-		)
-		(pin "13"
-		)
-		(pin "5"
-		)
-		(pin "12"
-		)
-		(pin "14"
-		)
-		(pin "4"
-		)
-		(pin "11"
-		)
-		(pin "16"
-		)
-		(pin "7"
-		)
-		(pin "9"
-		)
-		(pin "3"
-		)
-		(pin "1"
-		)
-		(pin "15"
-		)
-		(pin "2"
-		)
-		(pin "8"
-		)
-		(instances
-			(project "P1_Lock"
-				(path "/5e2df9ca-03bb-49be-9c86-c051a8edf5f2"
-					(reference "U2")
-					(unit 1)
-				)

Commit message: added keypad to library
Parts:
- removed J1: Conn_01x07, symbol Connector_Generic:Conn_01x07
- added SW1: ADA-419, symbol P1_SymbolLibrary:ADA-419
Connections:
- net at U1.21 (PA5): now also SW1.1 (COL1)
- net at U1.22 (PA6): now also SW1.2 (COL2)
- net at U1.23 (PA7): now also SW1.3 (COL3)
Changed lines of the file:
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@@
 	(wire
 		(pts
-			(xy 157.48 110.49) (xy 157.48 69.85)
+			(xy 157.48 111.76) (xy 157.48 69.85)
 		)
 		(stroke
@@
 	(wire
 		(pts
-			(xy 187.96 107.95) (xy 160.02 107.95)
+			(xy 191.77 109.22) (xy 160.02 109.22)
 		)
 		(stroke
@@
 	(wire
 		(pts
-			(xy 187.96 110.49) (xy 157.48 110.49)
+			(xy 191.77 111.76) (xy 157.48 111.76)
 		)
 		(stroke
@@
 	(wire
 		(pts
-			(xy 154.94 113.03) (xy 187.96 113.03)
+			(xy 154.94 114.3) (xy 191.77 114.3)
 		)
 		(stroke
@@
 	(wire
 		(pts
-			(xy 154.94 113.03) (xy 154.94 72.39)
+			(xy 154.94 114.3) (xy 154.94 72.39)
 		)
 		(stroke
@@
 	(wire
 		(pts
-			(xy 160.02 67.31) (xy 160.02 107.95)
+			(xy 160.02 67.31) (xy 160.02 109.22)
 		)
 		(stroke
@@
 	)
 	(symbol
-		(lib_id "Connector_Generic:Conn_01x07")
-		(at 193.04 115.57 0)
-		(unit 1)
-		(body_style 1)
-		(exclude_from_sim no)
-		(in_bom yes)
-		(on_board yes)
-		(in_pos_files yes)
-		(dnp no)
-		(fields_autoplaced yes)
-		(property "Reference" "J1"
-			(at 195.58 114.2999 0)
-			(show_name no)
-			(do_not_autoplace no)
-			(effects
-				(font
-					(size 1.27 1.27)
-				)
-				(justify left)
-			)
-		)
-		(property "Value" "Conn_01x07"
-			(at 195.58 116.8399 0)
-			(show_name no)
-			(do_not_autoplace no)
-			(effects
-				(font
-					(size 1.27 1.27)
-				)
-				(justify left)
-			)
-		)
-		(property "Footprint" ""
-			(at 193.04 115.57 0)
-			(hide yes)
-			(show_name no)
-			(do_not_autoplace no)
-			(effects
-				(font
-					(size 1.27 1.27)
-				)
-			)
-		)
-		(property "Datasheet" ""
-			(at 193.04 115.57 0)
-			(hide yes)
-			(show_name no)
-			(do_not_autoplace no)
-			(effects
-				(font
-					(size 1.27 1.27)
-				)
-			)
-		)
-		(property "Description" "Generic connector, single row, 01x07, script generated (kicad-library-utils/schlib/autogen/connector/)"
-			(at 193.04 115.57 0)
-			(hide yes)
-			(show_name no)
-			(do_not_autoplace no)
-			(effects
-				(font
-					(size 1.27 1.27)
-				)
-			)
-		)
-		(pin "1"
-		)
-		(pin "7"
-		)
-		(pin "4"
-		)
-		(pin "6"
-		)
-		(pin "3"
-		)
-		(pin "2"
-		)
-		(pin "5"
-		)
-		(instances
-			(project "P1_Lock"
-				(path "/5e2df9ca-03bb-49be-9c86-c051a8edf5f2"
-					(reference "J1")
-					(unit 1)
-				)
-			)
-		)
-	)
-	(symbol
 		(lib_id "P1_SymbolLibrary:QAPASS 1602A")
 		(at 198.12 71.12 0)
@@
 					(unit 1)
 				)
+			)
+		)
+	)
+	(symbol
+		(lib_id "P1_SymbolLibrary:ADA-419")
+		(at 207.01 116.84 0)
+		(unit 1)
+		(body_style 1)
+		(exclude_from_sim no)
+		(in_bom yes)
+		(on_board yes)
+		(in_pos_files yes)
+		(dnp no)
+		(fields_autoplaced yes)
+		(property "Reference" "SW1"
+			(at 219.71 115.5699 0)
+			(show_name no)
+			(do_not_autoplace no)
+			(effects
+				(font
+					(size 1.27 1.27)
+				)
+				(justify left)
+			)
+		)
+		(property "Value" "ADA-419"
+			(at 219.71 118.1099 0)
+			(show_name no)
+			(do_not_autoplace no)
+			(effects
+				(font
+					(size 1.27 1.27)
+				)
+				(justify left)
+			)
+		)
+		(property "Footprint" ""
+			(at 207.01 116.84 0)
+			(hide yes)
+			(show_name no)
+			(do_not_autoplace no)
+			(effects
+				(font
+					(size 1.27 1.27)
+				)
+			)
+		)
+		(property "Datasheet" ""
+			(at 207.01 116.84 0)
+			(hide yes)
+			(show_name no)
+			(do_not_autoplace no)
+			(effects
+				(font
+					(size 1.27 1.27)
+				)
+			)
+		)
+		(property "Description" "Generic connector, single row, 01x07, script generated (kicad-library-utils/schlib/autogen/connector/)"
+			(at 207.01 116.84 0)
+			(hide yes)
+			(show_name no)
+			(do_not_autoplace no)
+			(effects
+				(font
+					(size 1.27 1.27)
+				)
+			)
+		)
+		(pin "5"
+		)
+		(pin "2"
+		)
+		(pin "1"
+		)
+		(pin "3"
+		)
+		(pin "4"
+		)
+		(pin "6"
+		)
+		(pin "7"
+		)
+		(instances
+			(project "P1_Lock"
+				(path "/5e2df9ca-03bb-49be-9c86-c051a8edf5f2"
+					(reference "SW1")
+					(unit 1)
+				)
