File: hardware/P1_Lock.kicad_sch (KiCad schematic)
At the start: 6 parts, among them SW1 ADA-419, U1 STM32L476RGTx

Commit message: updated library symbols
Connections:
- net at U1.22 (PA6): now also SW1.2 (ROW2)
- net at U1.23 (PA7): now also SW1.3 (ROW3)
- net at U1.41 (PA8): now also SW1.4 (ROW4)
- net at U1.51 (PC10): now also SW1.5 (COL1)
- net at U1.52 (PC11): now also SW1.6 (COL2)
- net at U1.53 (PC12): now also SW1.7 (COL3)
Other:
- moved on the sheet: SW1
Changed lines of the file:
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@@
+	(wire
+		(pts
+			(xy 100.33 105.41) (xy 109.22 105.41)
+		)
+		(stroke
+			(width 0)
+			(type default)
+		)
+	)
 	(wire
 		(pts
@@
 	(wire
 		(pts
+			(xy 96.52 102.87) (xy 109.22 102.87)
+		)
+		(stroke
+			(width 0)
+			(type default)
+		)
+	)
+	(wire
+		(pts
 			(xy 102.87 57.15) (xy 102.87 44.45)
 		)
@@
 	(wire
 		(pts
+			(xy 100.33 160.02) (xy 100.33 105.41)
+		)
+		(stroke
+			(width 0)
+			(type default)
+		)
+	)
+	(wire
+		(pts
 			(xy 109.22 85.09) (xy 86.36 85.09)
 		)
@@
 	(wire
 		(pts
+			(xy 184.15 160.02) (xy 100.33 160.02)
+		)
+		(stroke
+			(width 0)
+			(type default)
+		)
+	)
+	(wire
+		(pts
+			(xy 187.96 123.19) (xy 187.96 162.56)
+		)
+		(stroke
+			(width 0)
+			(type default)
+		)
+	)
+	(wire
+		(pts
+			(xy 187.96 120.65) (xy 184.15 120.65)
+		)
+		(stroke
+			(width 0)
+			(type default)
+		)
+	)
+	(wire
+		(pts
 			(xy 91.44 80.01) (xy 91.44 72.39)
 		)
@@
 	(wire
 		(pts
+			(xy 104.14 107.95) (xy 109.22 107.95)
+		)
+		(stroke
+			(width 0)
+			(type default)
+		)
+	)
+	(wire
+		(pts
 			(xy 58.42 62.23) (xy 58.42 102.87)
 		)
@@
 	(wire
 		(pts
+			(xy 104.14 162.56) (xy 104.14 107.95)
+		)
+		(stroke
+			(width 0)
+			(type default)
+		)
+	)
+	(wire
+		(pts
 			(xy 102.87 44.45) (xy 119.38 44.45)
 		)
@@
 	(wire
 		(pts
+			(xy 180.34 118.11) (xy 180.34 156.21)
+		)
+		(stroke
+			(width 0)
+			(type default)
+		)
+	)
+	(wire
+		(pts
 			(xy 165.1 64.77) (xy 167.64 64.77)
 		)
@@
 	(wire
 		(pts
+			(xy 184.15 120.65) (xy 184.15 160.02)
+		)
+		(stroke
+			(width 0)
+			(type default)
+		)
+	)
+	(wire
+		(pts
 			(xy 157.48 110.49) (xy 157.48 69.85)
 		)
@@
 	(wire
 		(pts
+			(xy 187.96 118.11) (xy 180.34 118.11)
+		)
+		(stroke
+			(width 0)
+			(type default)
+		)
+	)
+	(wire
+		(pts
 			(xy 154.94 72.39) (xy 144.78 72.39)
 		)
@@
 	(wire
 		(pts
+			(xy 180.34 156.21) (xy 96.52 156.21)
+		)
+		(stroke
+			(width 0)
+			(type default)
+		)
+	)
+	(wire
+		(pts
 			(xy 109.22 97.79) (xy 73.66 97.79)
 		)
@@
 	(wire
 		(pts
+			(xy 96.52 156.21) (xy 96.52 102.87)
+		)
+		(stroke
+			(width 0)
+			(type default)
+		)
+	)
+	(wire
+		(pts
 			(xy 187.96 115.57) (xy 152.4 115.57)
+		)
+		(stroke
+			(width 0)
+			(type default)
+		)
+	)
+	(wire
+		(pts
+			(xy 187.96 162.56) (xy 104.14 162.56)
 		)
 		(stroke
@@
 	(symbol
 		(lib_id "P1_SymbolLibrary:ADA-419")
-		(at 207.01 116.84 0)
+		(at 203.2 115.57 0)
 		(unit 1)
 		(body_style 1)
@@
 		(fields_autoplaced yes)
 		(property "Reference" "SW1"
-			(at 219.71 115.5699 0)
+			(at 215.9 114.2999 0)
 			(show_name no)
 			(do_not_autoplace no)
@@
 		)
 		(property "Value" "ADA-419"
-			(at 219.71 118.1099 0)
+			(at 215.9 116.8399 0)
 			(show_name no)
 			(do_not_autoplace no)
@@
 		)
 		(property "Footprint" ""
-			(at 207.01 116.84 0)
+			(at 203.2 115.57 0)
 			(hide yes)
 			(show_name no)
@@
 		)
 		(property "Datasheet" ""
-			(at 207.01 116.84 0)
+			(at 203.2 115.57 0)
 			(hide yes)
 			(show_name no)
@@
 		)
 		(property "Description" "Generic connector, single row, 01x07, script generated (kicad-library-utils/schlib/autogen/connector/)"
-			(at 207.01 116.84 0)
-			(hide yes)
-			(show_name no)
+			(at 203.2 115.57 0)
+			(hide yes)
+			(show_name no)

Commit message: schematic finalized
Connections:
- net GNDREF: now reaches D1.1 (K), DS1.16 (K), DS1.2 (VDD), U1.18 (VSS), U1.31 (VSS), U1.47 (VSS), U1.63 (VSS)
- net +5V: now reaches DS1.1 (VSS), DS1.15 (A), RV1.3
- net +5V: no longer U1.65 (5V)
- net +3.3V: now reaches U1.19 (VDD)
